Commit message: modified frame for laser

File: urdf/accessories/sick_lms2xx.urdf.xacro (robot description, xacro)
@@ -12,5 +12,5 @@
       </inertial>
       <visual>
-        <origin xyz="0 0 0" rpy="0 0 0" />
+        <origin xyz="0 0 0" rpy="0 0 1.5708" />
         <geometry>
           <!-- Origin of this mesh is the focal point of the LIDAR. -->

File: urdf/husky.urdf.xacro (robot description, xacro)
@@ -41,4 +41,11 @@
   <xacro:arg name="laser_secondary_xyz"     default="$(optenv HUSKY_LMS1XX_SECONDARY_XYZ -0.2206 0.0 0.00635)" />
   <xacro:arg name="laser_secondary_rpy"     default="$(optenv HUSKY_LMS1XX_SECONDARY_RPY 0.0 0.0 3.14159)" />
+  <xacro:arg name="laser_lms2xx_secondary_enabled" default="$(optenv HUSKY_LMS2XX_SECONDARY_ENABLED 0)" />
+  <xacro:arg name="laser_lms2xx_secondary_topic"   default="$(optenv HUSKY_LMS2XX_SECONDARY_TOPIC front/scan)"/>
+  <xacro:arg name="laser_lms2xx_secondary_tower"   default="$(optenv HUSKY_LMS2XX_SECONDARY_TOWER 0)"/>
+  <xacro:arg name="laser_lms2xx_secondary_prefix"  default="$(optenv HUSKY_LMS2XX_SECONDARY_PREFIX rear)"/>
+  <xacro:arg name="laser_lms2xx_secondary_parent"  default="$(optenv HUSKY_LMS2XX_SECONDARY_PARENT base_link)"/>
+  <xacro:arg name="laser_lms2xx_secondary_xyz"     default="$(optenv HUSKY_LMS2XX_SECONDARY_XYZ -0.2206 0.0 0.00635)" />
+  <xacro:arg name="laser_lms2xx_secondary_rpy"     default="$(optenv HUSKY_LMS2XX_SECONDARY_RPY 0.0 0.0 3.14159)" />
   <!-- UST10 Laser Primary  and Secondary -->
   <xacro:arg name="laser_ust10_front_enabled" default="$(optenv HUSKY_UST10_ENABLED 0)" />
@@ -122,4 +129,5 @@
   <xacro:include filename="$(find husky_description)/urdf/accessories/sensor_arch.urdf.xacro"/>
   <xacro:include filename="$(find husky_description)/urdf/accessories/sick_lms1xx_mount.urdf.xacro"/>
+  <xacro:include filename="$(find husky_description)/urdf/accessories/sick_lms2xx.urdf.xacro"/>
   <xacro:include filename="$(find husky_description)/urdf/accessories/vlp16_mount.urdf.xacro"/>
   <xacro:include filename="$(find husky_description)/urdf/decorations.urdf.xacro" />
@@ -137,6 +145,10 @@
   <xacro:property name="wheel_length" value="0.1143" />
   <xacro:property name="wheel_radius" value="0.1651" />
+  <link name="base_link_rotated">
+    <origin xyz="0 0 0" rpy="0 0 0" />
+  </link>
   <!-- Base link is the center of the robot's bottom plate -->
   <link name="base_link">
+    <origin xyz="0 0 0" rpy="0 0 ${M_PI}" />
     <visual>
       <origin xyz="0 0 0" rpy="0 0 0" />
@@ -164,4 +176,9 @@
     <parent link="base_link" />
     <child link="base_footprint" />
+  </joint>
+  <joint name="base_rotate_joint" type="fixed">
+    <origin xyz="0 0 0" rpy="0 0 ${M_PI}" />
+    <parent link="base_link_rotated" />
+    <child link="base_link" />
   </joint>
   <!-- Inertial link stores the robot's inertial information -->
@@ -225,4 +242,16 @@
       <origin xyz="$(arg laser_secondary_xyz)" rpy="$(arg laser_secondary_rpy)"/>
     </xacro:sick_lms1xx_mount>
+  </xacro:if>
+  <!--
+    SICK LMS2XX Secondary Laser Scans
+  -->
+  <xacro:if value="$(arg laser_lms2xx_secondary_enabled)">
+    <xacro:sick_lms2xx  topic="$(arg laser_lms2xx_secondary_topic)" robot_namespace="$(arg robot_namespace)" />
+    <joint name="laser_joint" type="fixed">
+      <!-- This offset is from the base of the husky to the LIDAR's focal point. -->
+      <origin xyz="$(arg laser_lms2xx_secondary_xyz)" rpy="$(arg laser_lms2xx_secondary_rpy)"/>
+      <parent link="$(arg laser_lms2xx_secondary_parent)" />
+      <child link="laser" />
+    </joint>
   </xacro:if>
   <!--
